Commit message: slider control update

File: ros2_ws/install/robot_description/share/robot_description/urdf/common_properties.xacro (robot description, xacro)
@@ -1 +1,61 @@
-/home/raz/projects/astroscale/ros2_ws/src/robot_description/urdf/common_properties.xacro
+<?xml version="1.0"?>
+<robot xmlns:xacro="http://www.ros.org/wiki/xacro">
+    <!-- Common Constants -->
+    <xacro:property name="PI" value="3.141592653589793" />
+    <!-- Common Colors -->
+    <material name="black">
+        <color rgba="0.05 0.05 0.05 1" />
+    </material>
+    <material name="white">
+        <color rgba="0.9 0.9 0.9 1" />
+    </material>
+    <material name="silver">
+        <color rgba="0.75 0.75 0.75 1" />
+    </material>
+    <material name="red">
+        <color rgba="0.5 0 0 1" />
+    </material>
+    <material name="green">
+        <color rgba="0 0.5 0 1" />
+    </material>
+    <material name="blue">
+        <color rgba="0 0 0.5 1" />
+    </material>
+    <material name="grey">
+        <color rgba="0.5 0.5 0.5 1" />
+    </material>
+    <material name="orange">
+        <color rgba="1 0.65 0 1" />
+    </material>
+    <material name="yellow">
+        <color rgba="1 1 0 1" />
+    </material>
+    <!-- Common Momentun of Inertia -->
+    <xacro:macro name="box_inertia" params="m l w h xyz rpy">
+        <inertial>
+            <origin xyz="${xyz}" rpy="${rpy}" />
+            <mass value="${m}" />
+            <inertia ixx="${(m/12) * (h*h + l*l)}" ixy="0"                        ixz="0"
+                                                   iyy="${(m/12) * (w*w + l*l)}"  iyz="0"
+                                                                                  izz="${(m/12) * (w*w + h*h)}" />
+        </inertial>
+    </xacro:macro>
+    <xacro:macro name="cylinder_inertia" params="m r h xyz rpy">
+        <inertial>
+            <origin xyz="${xyz}" rpy="${rpy}" />
+            <mass value="${m}" />
+            <inertia ixx="${(1/12) * m * (3*r*r + h*h)}"  ixy="0"                              ixz="0"
+                                                          iyy="${(1/12) * m * (3*r*r + h*h)}"  iyz="0"
+                                                                                               izz="${(1/2) * m * (r*r)}" />
+        </inertial>
+    </xacro:macro>
+    <xacro:macro name="sphere_inertia" params="m r xyz rpy">
+        <inertial>
+            <origin xyz="${xyz}" rpy="${rpy}" />
+            <mass value="${m}" />
+            <inertia ixx="${(2/5) * m * (r*r)}"  ixy="0"                     ixz="0"
+                                                 iyy="${(2/5) * m * (r*r)}"  iyz="0"
+                                                                             izz="${(2/5) * m * (r*r)}" />
+        </inertial>
+    </xacro:macro>
+</robot>

File: ros2_ws/install/robot_description/share/robot_description/urdf/manipulator.urdf.xacro (robot description, xacro)
@@ -1 +1,77 @@
-/home/raz/projects/astroscale/ros2_ws/src/robot_description/urdf/manipulator.urdf.xacro
+<?xml version="1.0"?>
+<robot xmlns:xacro="http://www.ros.org/wiki/xacro" name="manipulator">
+    <!-- Include Common Properties -->
+    <xacro:include filename="common_properties.xacro" />
+    <!-- Include Gazebo Parameters -->
+    <xacro:include filename="$(find robot_description)/urdf/robot_gazebo.xacro" />
+    <!-- Include Ros2 Control Parameters -->
+    <xacro:include filename="$(find robot_description)/urdf/robot_ros2_control.xacro" />
+    <!-- Useful XACRO Variables (Properties) -->
+    <xacro:property name="effort" value="30.0" />
+    <xacro:property name="velocity" value="10.0" />
+    <!-- Dimensions -->
+    <xacro:property name="arm_base_length" value="0.15" />
+    <xacro:property name="arm_base_height" value="0.03" />
+    <xacro:property name="arm_radius" value="0.02" />
+    <xacro:property name="arm_length" value="0.3" />
+    <!-- Links -->
+    <link name="world" />
+    <link name="base_link">
+        <visual>
+            <geometry>
+                <box size="${arm_base_length} ${arm_base_length} ${arm_base_height}" />
+            </geometry>
+            <origin xyz="0 0 ${arm_base_height / 2.0}" rpy="0 0 0" />
+            <material name="white" />
+        </visual>
+        <collision>
+            <geometry>
+                <box size="${arm_base_length} ${arm_base_length} ${arm_base_height}" />
+            </geometry>
+            <origin xyz="0 0 ${arm_base_height / 2.0}" rpy="0 0 0" />
+        </collision>
+        <xacro:box_inertia m="1" l="${arm_base_length}" w="${arm_base_length}" h="${arm_base_height}"
+                           xyz="0 0 ${arm_base_height / 2.0}" rpy="0 0 0" />
+    </link>
+    <xacro:macro name="arm_link" params="prefix color">
+        <link name="${prefix}_link">
+            <visual>
+                <geometry>
+                    <cylinder radius="${arm_radius}" length="${arm_length}" />
+                </geometry>
+                <origin xyz="0 0 ${arm_length / 2.0}" rpy="0 0 0" />
+                <material name="${color}" />
+            </visual>
+            <collision>
+                <geometry>
+                    <cylinder radius="${arm_radius}" length="${arm_length}" />
+                </geometry>
+                <origin xyz="0 0 ${arm_length / 2.0}" rpy="0 0 0" />
+            </collision>
+            <xacro:cylinder_inertia m="0.3" r="${arm_radius}" h="${arm_length}"
+                                    xyz="0 0 ${arm_length / 2.0}" rpy="0 0 0" />
+        </link>
+    </xacro:macro>
+    <xacro:arm_link prefix="forearm" color="black" />
+    <xacro:arm_link prefix="hand" color="silver" />
+    <!-- Joints -->
+    <joint name="virtual_joint" type="fixed">
+        <parent link="world" />
+        <child link="base_link" />
+        <origin xyz="0 0 0" rpy="0 0 0" />
+    </joint>
+    <joint name="joint1" type="revolute">
+        <parent link="base_link" />
+        <child link="forearm_link" />
+        <origin xyz="0 0 ${arm_base_height}" rpy="0 0 0" />
+        <axis xyz="0 0 1" />
+        <limit lower="-${PI}" upper="${PI}" effort="${effort}" velocity="${velocity}" />
+    </joint>
+    <joint name="joint2" type="revolute">
+        <parent link="forearm_link" />
+        <child link="hand_link" />
+        <origin xyz="0 0 ${arm_length}" rpy="0 0 0" />
+        <axis xyz="0 1 0" />
+        <limit lower="-${PI / 2.0}" upper="${PI / 2.0}" effort="${effort}" velocity="${velocity}" />
+    </joint>
+</robot>

File: ros2_ws/install/robot_description/share/robot_description/urdf/robot_gazebo.xacro (robot description, xacro)
@@ -1 +1,9 @@
-/home/raz/projects/astroscale/ros2_ws/src/robot_description/urdf/robot_gazebo.xacro
+<?xml version="1.0"?>
+<robot xmlns:xacro="http://www.ros.org/wiki/xacro" name="manipuator">
+    <!-- Gazebo Control Plugin -->
+    <gazebo>
+        <plugin filename="ign_ros2_control-system" name="ign_ros2_control::IgnitionROS2ControlPlugin">
+            <parameters>$(find robot_controller)/config/robot_controllers.yaml</parameters>
+        </plugin>
+    </gazebo>
+</robot>

File: ros2_ws/install/robot_description/share/robot_description/urdf/robot_ros2_control.xacro (robot description, xacro)
@@ -1 +1,23 @@
-/home/raz/projects/astroscale/ros2_ws/src/robot_description/urdf/robot_ros2_control.xacro
+<?xml version="1.0"?>
+<robot xmlns:xacro="http://www.ros.org/wiki/xacro" name="manipulator">
+    <ros2_control name="RobotSystem" type="system">
+        <!-- ros2 control Gazebo -->
+        <hardware>
+            <plugin>ign_ros2_control/IgnitionSystem</plugin>
+        </hardware>
+        <joint name="joint1">
+            <command_interface name="position">
+            <param name="min">-${PI}</param>
+            <param name="max">${PI}</param>
+            </command_interface>
+            <state_interface name="position"/>
+        </joint>
+        <joint name="joint2">
+            <command_interface name="position">
+            <param name="min">-${PI / 2.0}</param>
+            <param name="max">${PI / 2.0}</param>
+            </command_interface >
+            <state_interface name="position"/>
+        </joint>
+    </ros2_control>
+</robot>
